Commit message: update h joint limit

File: urdf/five_dof_arm.urdf (robot description, URDF)
Before this commit: robot five_dof_arm, 7 links, 6 joints
Joints:
- joint joint_5: limit lower=-3.14159265359 upper=3.14159265359 effort=10 velocity=2 -> lower=-0.785398163397 upper=0.785398163397 effort=10 velocity=2

Commit message: corrected kinematics

File: urdf/five_dof_arm.urdf (robot description, URDF)
Before this commit: robot five_dof_arm, 7 links, 6 joints
Joints:
- joint joint_1: axis 0 0 -1 -> 0 0 1
- joint joint_2: axis 0 0 -1 -> 0 0 1; limit lower=-3.14159265359 upper=3.14159265359 effort=10 velocity=2 -> lower=-1.57079632679 upper=1.57079632679 effort=10 velocity=2; origin xyz=0 0 0.0335 rpy=1.57079632679 0 0 -> xyz=0 0 0.0335 rpy=-1.57079632679 0 0
- joint joint_3: axis 0 0 -1 -> 0 0 1; limit lower=-3.14159265359 upper=3.14159265359 effort=10 velocity=2 -> lower=-1.57079632679 upper=1.57079632679 effort=10 velocity=2; origin xyz=0.03564 0.23002 0 rpy=0 0 0 -> xyz=0.03564 -0.23002 0 rpy=0 0 0
- joint joint_4: axis 0 0 1 -> 0 0 -1; limit lower=-3.14159265359 upper=3.14159265359 effort=10 velocity=2 -> lower=-1.57079632679 upper=1.57079632679 effort=10 velocity=2; origin xyz=0.24164 0 0 rpy=0 -1.57079632679 3.14159265359 -> xyz=0.24164 0 0 rpy=0 -1.57079632679 -3.14159265359
- joint joint_5: axis 0 0 1 -> 0 0 -1; origin xyz=0.0121 -0.02478 0.01835 rpy=0 -1.57079632679 1.57079632679 -> xyz=0.0121 0.02478 0.01835 rpy=0 -1.57079632679 -1.57079632679
- joint pen_tip_fixed_joint: origin xyz=0.03431 -0.08012 -0.02672 rpy=-1.57079632679 0 0 -> xyz=0.03431 0.08012 -0.02672 rpy=1.57079632679 0 0

Commit message: modified pen's location

File: urdf/five_dof_arm.urdf (robot description, URDF)
Before this commit: robot five_dof_arm, 7 links, 6 joints
Links:
- added link nib_marker; visual sphere radius=0.006
- added link tail_marker; visual sphere radius=0.006
Joints:
- added joint nib_marker_fixed: type fixed, parent link_5, child nib_marker, origin xyz=0.04473864 -0.07941421 0.030 rpy=0 0 0
- added joint tail_marker_fixed: type fixed, parent link_5, child tail_marker, origin xyz=0.02646136 0.03921421 0.030 rpy=0 0 0

Commit message: updated kinematics

File: urdf/five_dof_arm.urdf (robot description, URDF)
Before this commit: robot five_dof_arm, 9 links, 8 joints
Joints:
- joint nib_marker_fixed: origin xyz=0.04473864 -0.07941421 0.030 rpy=0 0 0 -> xyz=0.0508886 -0.07813403 0.030 rpy=0 0 0
- joint tail_marker_fixed: origin xyz=0.02646136 0.03921421 0.030 rpy=0 0 0 -> xyz=0.0203114 0.03793403 0.030 rpy=0 0 0
